Commit message: Update trucon robot URDF

File: src/trucon_description/urdf/trucon_robot.urdf (robot description, URDF)
Before this commit: robot trucon_robot, 6 links, 5 joints
Links:
- added link left_wheel_link, mass 0.3; collision cylinder length=0.04 radius=0.05; visual cylinder length=0.04 radius=0.05
- added link right_wheel_link, mass 0.3; collision cylinder length=0.04 radius=0.05; visual cylinder length=0.04 radius=0.05
Joints:
- added joint left_wheel_joint: type continuous, parent base_link, child left_wheel_link, origin xyz=-0.1 0.0 -0.1 rpy=0 1.5708 0, axis 0 0 1
- added joint right_wheel_joint: type continuous, parent base_link, child right_wheel_link, origin xyz=0.1 0 -0.1 rpy=0 1.5708 0, axis 0 1 0
