Commit message: Week2 Monday: gripper URDF, ros2_control, joint_state_broadcaster, gripper open/close demo

File: src/trucon_description/urdf/trucon_robot.urdf (robot description, URDF)
Before this commit: robot trucon_robot, 8 links, 7 joints
Links:
- added link gripper_base_link, mass 0.1; collision box size=0.04 0.06 0.02; visual box size=0.04 0.06 0.02
- added link gripper_left_finger_link, mass 0.02; collision box size=0.01 0.02 0.04; visual box size=0.01 0.02 0.04
- added link gripper_right_finger_link, mass 0.02; collision box size=0.01 0.02 0.04; visual box size=0.01 0.02 0.04
Joints:
- added joint gripper_base_joint: type fixed, parent right_arm_link, child gripper_base_link, origin xyz=0 0 -0.15 rpy=0 0 0
- added joint gripper_left_finger_joint: type prismatic, parent gripper_base_link, child gripper_left_finger_link, origin xyz=0 0.02 -0.02 rpy=0 0 0, axis 0 1 0, limit lower=0 upper=0.03 effort=5 velocity=0.1
- added joint gripper_right_finger_joint: type prismatic, parent gripper_base_link, child gripper_right_finger_link, origin xyz=0 -0.02 -0.02 rpy=0 0 0, axis 0 -1 0, limit lower=0 upper=0.03 effort=5 velocity=0.1
